Commit message: 修改了日志存储器,修改了存放位置

File: src/usv_simulation/vrx/vrx_urdf/wamv_description/urdf/wamv_base.urdf.xacro (robot description, xacro)
@@ -88,8 +88,8 @@
     <visual>
       <geometry>
-        <mesh filename="package://wamv_description/models/WAM-V-Base/mesh/M5_body.dae"/>
+        <mesh filename="package://wamv_description/models/WAM-V-Base/mesh/WAM-V-Base.dae"/>
       </geometry>
     </visual>
-    <!-- <mesh filename="package://wamv_description/models/WAM-V-Base/mesh/WAM-V-Base.dae"/> -->
+    <!-- <mesh filename="package://wamv_description/models/WAM-V-Base/mesh/blade_R.dae"/> -->
 <!-- src/my_wamv/blade_R.dae -->
     <!-- Left base collisions -->

Commit message: 调整了模型映射路径,重新设置了xacro文件

File: src/usv_simulation/vrx/vrx_urdf/wamv_description/urdf/wamv_base.urdf.xacro (robot description, xacro)
@@ -4,4 +4,6 @@
   <xacro:arg name="namespace" default="wamv"/>
   <xacro:property name="namespace" value="$(arg namespace)" scope="global" />
+  <!-- Visual mesh argument -->
+  <xacro:arg name="visual_mesh" default="package://wamv_description/models/WAM-V-Base/mesh/WAM-V-Base.dae"/>
   <!-- Macro for creating the main collisions as simple shapes. -->
   <xacro:macro name="main_collisions" params="prefix reflect:=1">
@@ -88,5 +90,5 @@
     <visual>
       <geometry>
-        <mesh filename="package://wamv_description/models/WAM-V-Base/mesh/WAM-V-Base.dae"/>
+        <mesh filename="$(arg visual_mesh)"/>
       </geometry>
     </visual>
